File: PCB/Nif-T.kicad_sch (KiCad schematic)
At the start: 0 parts

Commit message: Big ol trip
Worked on this while traveling.
Parts:
- added C1, C2, C3: 0.22uF, imported_components:C0805, symbol Device:C
- added C10, C13, C4, C5, C7, C9: 0.1uF, imported_components:C0805, symbol Device:C
- added C11, C6, C8: 1uF, imported_components:C0805, symbol Device:C
- added C12: 10uF, imported_components:C0805, symbol Device:C
- added D1: SS54_C22452, imported_components:SMA_L4.4-W2.8-LS5.4-R-RD, symbol imported_components:SS54_C22452
- added FB1: FerriteBead, symbol Device:FerriteBead
- added P1: USB_C_Plug, imported_components:USB-C_SMD-TYPE-C-31-M-12, symbol Connector:USB_C_Plug
- added R1: 12.1k, imported_components:R0805, symbol Device:R
- added R10, R11, R12, R13, R3: 10k, imported_components:R0805, symbol Device:R
- added R2: 22, imported_components:R0805, symbol Device:R
- added R4, R5, R6, R7: 49.9, imported_components:R0805, symbol Device:R
- added R8, R9: 5.1k, imported_components:R0805, symbol Device:R
- added RJ1: HY931147C, new_imported_components:RJ45-TH_HY931147C, symbol new_imported_components:HY931147C
- added SW1, SW2: SW_Push, imported_components:SW-SMD_L3.9-W3.0-P4.45, symbol Switch:SW_Push
- added U1: ESP32-WROOM-32E(4MB), new_imported_components:WIFI-SMD_ESP32-WROOM-32E, symbol new_imported_components:ESP32-WROOM-32E(4MB)
- added U2: LAN8720A-CP-TR, new_imported_components:QFN-24_L4.0-W4.0-P0.50-BL-EP2.6, symbol new_imported_components:LAN8720A-CP-TR
- added U3: DP1435-5V, new_imported_components:PWRM-TH_DP1435-XX, symbol new_imported_components:DP1435-5V
- added U4: CH340C, Package_SO:SOIC-16_3.9x9.9mm_P1.27mm, symbol Interface_USB:CH340C
- added X1: X322525MOB4SI, new_imported_components:CRYSTAL-SMD_4P-L3.2-W2.5-BL, symbol new_imported_components:X322525MOB4SI
Connections:
- new net: R2.1, U2.14 (nINT/REFCLKO)
- new net: R1.1, U2.24 (RBIAS)
- new net: D1.1 (A), U3.6 (+5V)
- new net: P1.B5 (VCONN), R8.2
- new net: P1.A5 (CC), R9.1
- new net +3.3V: C12.2, C13.2, C4.1, FB1.1, R10.1, R11.1, R12.1, R13.2, R3.2, U1.2 (3V3), U4.16 (VCC), U4.4 (V3)
- new net +5V: D1.2 (K)
- new net 8720RST: R13.1, U1.29 (IO5), U2.15 (nRST)
- new net CHIP_PU: C10.1, C11.1, R11.2, R12.2, SW2.1, U1.3 (EN)
- new net CRS_DV/MODE2: U1.12 (IO27), U2.11 (CRS_DV/MODE2)
- new net ETH_CLK: C9.1, R10.2, R2.2, R3.1, SW1.1, U1.25 (IO0)
- new net GND: C1.2, C10.2, C11.2, C12.1, C13.1, C2.2, C3.1, C4.2, C5.2, C6.2, C7.2, C8.2, C9.2, P1.A1 (GND), P1.A12 (GND), P1.B1 (GND), P1.B12 (GND), P1.S1 (SHIELD), R1.2, R8.1, R9.2, RJ1.12, RJ1.14, RJ1.GND1 (GND), RJ1.GND2 (GND), SW1.2, SW2.2, U1.1 (GND), U1.15 (GND), U1.38 (GND), U1.39 (GND), U2.25 (EP), U3.5 (GND), U4.1 (GND), X1.2 (GND), X1.4 (GND)
- new net MDC: U1.37 (IO23), U2.13 (MDC)
- new net MDIO: U1.30 (IO18), U2.12 (MDIO)
- new net RJ45_LED_G: RJ1.13, U2.3 (LED1/REGOFF)
- new net RJ45_LED_Y: RJ1.11, U2.2 (LED2/nINTSEL)
- new net RJ45_V+: RJ1.9, U3.3 (VB1)
- new net RJ45_V-: RJ1.10, U3.4 (VB2)
- new net RX+: R6.1, RJ1.2, U2.23 (RXP)
- new net RX-: R7.1, RJ1.1, U2.22 (RXN)
- new net RXD0/MODE0: U1.10 (IO25), U2.8 (RXD0/MODE0)
- new net RXD1/MODE1: U1.11 (IO26), U2.7 (RXD1/MODE1)
- new net RX_CT: RJ1.3
- new net RX_P3: C1.1, C5.1, C6.1, C7.1, C8.1, FB1.2, R4.1, R5.2, R6.2, R7.2, U2.1 (VDD2A), U2.19 (VDD1A)
- new net TX+: R5.1, RJ1.6, U2.21 (TXP)
- new net TX-: R4.2, RJ1.5, U2.20 (TXN)
- new net TXD0: U1.31 (IO19), U2.17 (TXD0)
- new net TXD1: U1.36 (IO22), U2.18 (TXD1)
- new net TXEN: U1.33 (IO21), U2.16 (TXEN)
- new net TX_CT: RJ1.4
- new net USB_D+: P1.A6 (D+), U4.5 (UD+)
- new net USB_D-: P1.A7 (D-), U4.6 (UD-)
- new net USB_RX: U1.35 (TXD0), U4.3 (RXD)
- new net USB_TX: U1.34 (RXD0), U4.2 (TXD)
- new net VCC_5V: P1.A4 (VBUS), P1.A9 (VBUS), P1.B4 (VBUS), P1.B9 (VBUS)
- new net VDDCR: U2.6 (VDDCR)
- new net VDDIO: U2.9 (VDDIO)
- new net XTAL1: C3.2, U2.5 (XTAL1/CLKIN), X1.1 (OSC1)
- new net XTAL2: C2.1, U2.4 (XTAL2), X1.3 (OSC2)
- no-connect marks 0 -> 29
Other:
- added sheet POWER + IO (Nif-T_power_and_IO.kicad_sch)
- note added: "BOOT"
- note added: "BUTTONS"
- note added: "ESP32-WROOM-32E"
- note added: "ETHERNET"
- note added: "RST"
- note added: "USB-C"

Commit message: PCB Reconfigured and Rerouted
Parts:
- removed FB1: FerriteBead, symbol Device:FerriteBead
- added L2: BLM21PG221SN1D, new_imported_components:L0805, symbol new_imported_components:BLM21PG221SN1D
Connections:
- net VCC_5V is gone; now on net +5V: P1.A4 (VBUS), P1.A9 (VBUS), P1.B4 (VBUS), P1.B9 (VBUS)
- net +3.3V: now also L2.2
- net RX_CT: now also C1.1, C5.1, C6.1, C7.1, C8.1, R4.2, R5.2, R6.2, R7.2, U2.1 (VDD2A), U2.19 (VDD1A), L2.1
- net TX+: now also R4.1; no longer R5.1
- net TX-: now also R5.1; no longer R4.2
- net GPIO 14: now reaches U1.13 (IO14)
- net GPIO 13: now reaches U1.16 (IO13)
- net GPIO 15: now reaches U1.23 (IO15)
- net GPIO 2: now reaches U1.24 (IO2)
- net GPIO 4: now reaches U1.26 (IO4)
- net GPIO 16: now reaches U1.27 (IO16)
- net GPIO 17: now reaches U1.28 (IO17)
- net GPIO 36: now reaches U1.4 (SENSOR_VP)
- net GPIO 37: now reaches U1.5 (SENSOR_VN)
- net GPIO 34: now reaches U1.6 (IO34)
- net GPIO 35: now reaches U1.7 (IO35)
- net GPIO 32: now reaches U1.8 (IO32)
- net GPIO 33: now reaches U1.9 (IO33)
- removed net RX_P3: C1.1, C5.1, C6.1, C7.1, C8.1, R4.1, R5.2, R6.2, R7.2, U2.1 (VDD2A), U2.19 (VDD1A)
- net USB_RX renamed USB_UART-
- net USB_TX renamed USB_UART+
- no-connect marks 29 -> 30
Other:
- moved on the sheet: R4, R6, R7
