File: PCB/Nif-T_power_and_IO.kicad_sch (KiCad schematic)
At the start: 68 parts, among them J1 Barrel_Jack, J2 Conn_01x02, J3 Conn_02x03_Odd_Even, J4 Conn_02x03_Odd_Even, J5 Conn_02x03_Odd_Even, J6 Conn_02x03_Odd_Even, J7 Conn_02x03_Odd_Even, Q1 S8050, Q2 S8050, Q3 S8050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

Commit message: PCB Reconfigured and Rerouted
Parts:
- removed SW5: SW_DIP_x09, symbol Switch:SW_DIP_x09
- added D22: SS54_C22452, imported_components:SMA_L4.4-W2.8-LS5.4-R-RD, symbol imported_components:SS54_C22452
- added SW5, SW6: DSIC-05-LS-GER, new_imported_components:SW-SMD_DSIC-05-LS-GER, symbol new_imported_components:DSIC-05-LS-GER
Connections:
- net +5V: now also D22.2 (K); no longer C17.1, C19.1, L1.2, U5.4 (FB)
- net BUZZER_DATA: now also SW5.8
- net GPIO 13: now also SW6.5
- net GPIO 14: now also SW6.7
- net GPIO 15: now also SW5.3
- net GPIO 16: now also SW5.5, SW5.7
- net GPIO 17: now also SW5.9; no longer D4.2 (DIN)
- net GPIO 2: now also SW6.9
- net GPIO 32: now also SW6.1
- net GPIO 33: now also SW6.3
- net GPIO 4: now also SW5.1
- net RLY1CTRL: now also SW6.2
- net RLY2CTRL: now also SW6.4
- net RLY3CTRL: now also SW6.6
- net RLY4CTRL: now also SW6.8
- net RLY5CTRL: now also SW6.10
- net RLY6CTRL: now also SW5.2
- net RLY7CTRL: now also SW5.4
- net RLY8CTRL: now also SW5.6
- new net: C17.1, C19.1, D22.1 (A), L1.2, U5.4 (FB)
- new net LED_DATA: D4.2 (DIN), SW5.10
